Commit message: Rebase from 'upstream'

File: kuka_agilus_support/urdf/kr10_r1100_2.urdf.xacro (robot description, xacro)
@@ -3,9 +3,14 @@
   <!-- Import urdf file  -->
   <xacro:include filename="$(find kuka_agilus_support)/urdf/kr10_r1100_2_macro.xacro"/>
+  <xacro:include filename="$(find kuka_agilus_support)/urdf/kr_agilus_ros2_control_macro.xacro"/>
   <!-- Read additional arguments  -->
-  <xacro:arg name="use_fake_hardware" default="false"/>
+  <xacro:arg name="driver_version" default="rsi_only"/>
+  <xacro:arg name="mode" default="hardware"/>
+  <xacro:arg name="use_gpio" default="false"/>
   <xacro:arg name="roundtrip_time" default="0"/>
   <xacro:arg name="client_ip" default="0.0.0.0"/>
   <xacro:arg name="client_port" default="59152"/>
+  <xacro:arg name="controller_ip" default="0.0.0.0"/>
+  <xacro:arg name="verify_robot_model" default="true"/>
   <xacro:arg name="prefix" default=""/>
   <xacro:arg name="x" default="0"/>
@@ -15,5 +20,6 @@
   <xacro:arg name="pitch" default="0"/>
   <xacro:arg name="yaw" default="0"/>
-  <xacro:kuka_kr10_r1100_2_robot client_ip="$(arg client_ip)" client_port="$(arg client_port)" prefix="$(arg prefix)" use_fake_hardware="$(arg use_fake_hardware)" roundtrip_time="$(arg roundtrip_time)">
+  <xacro:kuka_agilus_ros2_control name="$(arg prefix)kr10_r1100_2" driver_version="$(arg driver_version)" client_ip="$(arg client_ip)" client_port="$(arg client_port)" controller_ip="$(arg controller_ip)" prefix="$(arg prefix)" mode="$(arg mode)" use_gpio="$(arg use_gpio)" roundtrip_time="$(arg roundtrip_time)" verify_robot_model="$(arg verify_robot_model)"/>
+  <xacro:kuka_kr10_r1100_2_robot prefix="$(arg prefix)" package_name="kuka_agilus_support">
     <origin xyz="$(arg x) $(arg y) $(arg z)" rpy="$(arg roll) $(arg pitch) $(arg yaw)"/>
   </xacro:kuka_kr10_r1100_2_robot>

File: kuka_agilus_support/urdf/kr10_r1100_2_macro.xacro (robot description, xacro)
@@ -2,10 +2,6 @@
 <robot xmlns:xacro="http://www.ros.org/wiki/xacro" name="kr10_r1100_2">
   <!-- include helper xacros -->
-  <xacro:include filename="$(find kuka_agilus_support)/urdf/kr_agilus_ros2_control.xacro"/>
-  <xacro:include filename="$(find kuka_agilus_support)/urdf/kr_agilus_transmission.xacro"/>
   <xacro:include filename="$(find kuka_resources)/urdf/common_materials.xacro"/>
-  <xacro:macro name="kuka_kr10_r1100_2_robot" params="client_ip client_port prefix use_fake_hardware roundtrip_time *origin">
-    <!-- ros2 control instance -->
-    <xacro:kuka_agilus_ros2_control name="${prefix}kr10_r1100_2" client_ip="${client_ip}" client_port="${client_port}" prefix="${prefix}" use_fake_hardware="${use_fake_hardware}" roundtrip_time="${roundtrip_time}"/>
+  <xacro:macro name="kuka_kr10_r1100_2_robot" params="prefix package_name *origin">
     <!-- links - main serial chain -->
     <link name="world"/>
@@ -13,11 +9,16 @@
       <collision>
         <geometry>
-          <mesh filename="package://kuka_agilus_support/meshes/kr10_r1100_2/collision/base_link.stl"/>
-        </geometry>
-        <origin rpy="-0.0 0.0 -0.0" xyz="0.0 0.0 0.0"/>
-      </collision>
-      <visual>
-        <geometry>
-          <mesh filename="package://kuka_agilus_support/meshes/kr10_r1100_2/visual/base_link.stl"/>
+          <mesh filename="package://${package_name}/meshes/kr10_r1100_2/collision/base_link.stl"/>
+        </geometry>
+        <origin rpy="-0.0 0.0 -0.0" xyz="0.0 0.0 0.0"/>
+      </collision>
+      <inertial>
+        <inertia ixx="0.16209200415615" ixy="0.0" ixz="0.0" iyy="0.10881181598555635" iyz="0.0" izz="0.18461591505869543"/>
+        <mass value="1.6916E1"/>
+        <origin rpy="1.6165592773339865 -1.221289277333065 3.10031147437779" xyz="-0.03713348309292976 2.6602033577676952E-5 0.10863850792149446"/>
+      </inertial>
+      <visual>
+        <geometry>
+          <mesh filename="package://${package_name}/meshes/kr10_r1100_2/visual/base_link.stl"/>
         </geometry>
         <origin rpy="-0.0 0.0 -0.0" xyz="0.0 0.0 0.0"/>
@@ -28,11 +29,16 @@
       <collision>
         <geometry>
-          <mesh filename="package://kuka_agilus_support/meshes/kr10_r1100_2/collision/link_1.stl"/>
-        </geometry>
-        <origin rpy="-0.0 0.0 -0.0" xyz="0.0 0.0 0.0"/>
-      </collision>
-      <visual>
-        <geometry>
-          <mesh filename="package://kuka_agilus_support/meshes/kr10_r1100_2/visual/link_1.stl"/>
+          <mesh filename="package://${package_name}/meshes/kr10_r1100_2/collision/link_1.stl"/>
+        </geometry>
+        <origin rpy="-0.0 0.0 -0.0" xyz="0.0 0.0 0.0"/>
+      </collision>
+      <inertial>
+        <inertia ixx="0.07406183855390855" ixy="0.0" ixz="0.0" iyy="0.0890478351825312" iyz="0.0" izz="0.11039570662759429"/>
+        <mass value="8.4159999999999986E0"/>
+        <origin rpy="1.304519343134156 -0.9428616016893947 -1.4226510948637578" xyz="0.006410408745247152 -0.01626805370722434 -0.10658893773764262"/>
+      </inertial>
+      <visual>
+        <geometry>
+          <mesh filename="package://${package_name}/meshes/kr10_r1100_2/visual/link_1.stl"/>
         </geometry>
         <origin rpy="-0.0 0.0 -0.0" xyz="0.0 0.0 0.0"/>
@@ -43,11 +49,16 @@
       <collision>
         <geometry>
-          <mesh filename="package://kuka_agilus_support/meshes/kr10_r1100_2/collision/link_2.stl"/>
-        </geometry>
-        <origin rpy="-0.0 0.0 -0.0" xyz="0.0 0.0 0.0"/>
-      </collision>
-      <visual>
-        <geometry>
-          <mesh filename="package://kuka_agilus_support/meshes/kr10_r1100_2/visual/link_2.stl"/>
+          <mesh filename="package://${package_name}/meshes/kr10_r1100_2/collision/link_2.stl"/>
+        </geometry>
+        <origin rpy="-0.0 0.0 -0.0" xyz="0.0 0.0 0.0"/>
+      </collision>
+      <inertial>
+        <inertia ixx="0.8751595055066254" ixy="0.0" ixz="0.0" iyy="0.09215049446198915" iyz="0.0" izz="0.9157117764876721"/>
+        <mass value="1.78369E1"/>
+        <origin rpy="1.9524873827550635 -1.5422358773344043 -0.3902815673307173" xyz="0.191160133767639 -0.004651344123698628 -0.07520541854245974"/>
+      </inertial>
+      <visual>
+        <geometry>
+          <mesh filename="package://${package_name}/meshes/kr10_r1100_2/visual/link_2.stl"/>
         </geometry>
         <origin rpy="-0.0 0.0 -0.0" xyz="0.0 0.0 0.0"/>
@@ -58,11 +69,16 @@
       <collision>
         <geometry>
-          <mesh filename="package://kuka_agilus_support/meshes/kr10_r1100_2/collision/link_3.stl"/>
-        </geometry>
-        <origin rpy="-0.0 0.0 -0.0" xyz="0.0 0.0 0.0"/>
-      </collision>
-      <visual>
-        <geometry>
-          <mesh filename="package://kuka_agilus_support/meshes/kr10_r1100_2/visual/link_3.stl"/>
+          <mesh filename="package://${package_name}/meshes/kr10_r1100_2/collision/link_3.stl"/>
+        </geometry>
+        <origin rpy="-0.0 0.0 -0.0" xyz="0.0 0.0 0.0"/>
+      </collision>
+      <inertial>
+        <inertia ixx="0.04469381119929391" ixy="0.0" ixz="0.0" iyy="0.018969508933922696" iyz="0.0" izz="0.0498412586885908"/>
+        <mass value="6.075E0"/>
+        <origin rpy="-2.676930368410595 -1.321895859309871 1.1860920267202666" xyz="0.04386106995884774 -0.012506995884773664 -0.06825142386831277"/>
+      </inertial>
+      <visual>
+        <geometry>
+          <mesh filename="package://${package_name}/meshes/kr10_r1100_2/visual/link_3.stl"/>
         </geometry>
         <origin rpy="-0.0 0.0 -0.0" xyz="0.0 0.0 0.0"/>
@@ -73,11 +89,16 @@
       <collision>
         <geometry>
-          <mesh filename="package://kuka_agilus_support/meshes/kr10_r1100_2/collision/link_4.stl"/>
-        </geometry>
-        <origin rpy="-0.0 0.0 -0.0" xyz="0.0 0.0 0.0"/>
-      </collision>
-      <visual>
-        <geometry>
-          <mesh filename="package://kuka_agilus_support/meshes/kr10_r1100_2/visual/link_4.stl"/>
+          <mesh filename="package://${package_name}/meshes/kr10_r1100_2/collision/link_4.stl"/>
+        </geometry>
+        <origin rpy="-0.0 0.0 -0.0" xyz="0.0 0.0 0.0"/>
+      </collision>
+      <inertial>
+        <inertia ixx="0.012301413884477554" ixy="0.0" ixz="0.0" iyy="0.08469612193319441" iyz="0.0" izz="0.08739834186747329"/>
+        <mass value="5.1623807059999995E0"/>
+        <origin rpy="-2.228094247436686 -1.5326119469267911 2.179783954730353" xyz="0.0013191433102012267 0.008607757626765767 -0.14098161935749579"/>
+      </inertial>
+      <visual>
+        <geometry>
+          <mesh filename="package://${package_name}/meshes/kr10_r1100_2/visual/link_4.stl"/>
         </geometry>
         <origin rpy="-0.0 0.0 -0.0" xyz="0.0 0.0 0.0"/>
@@ -88,11 +109,16 @@
       <collision>
         <geometry>
-          <mesh filename="package://kuka_agilus_support/meshes/kr10_r1100_2/collision/link_5.stl"/>
-        </geometry>
-        <origin rpy="-0.0 0.0 -0.0" xyz="0.0 0.0 0.0"/>
-      </collision>
-      <visual>
-        <geometry>
-          <mesh filename="package://kuka_agilus_support/meshes/kr10_r1100_2/visual/link_5.stl"/>
+          <mesh filename="package://${package_name}/meshes/kr10_r1100_2/collision/link_5.stl"/>
+        </geometry>
+        <origin rpy="-0.0 0.0 -0.0" xyz="0.0 0.0 0.0"/>
+      </collision>
+      <inertial>
+        <inertia ixx="0.0017317756133102904" ixy="0.0" ixz="0.0" iyy="0.002219500805440681" iyz="0.0" izz="0.002467090055442975"/>
+        <mass value="1.6128E0"/>
+        <origin rpy="1.567898714902774 -0.8611716764868309 -3.100280255900493" xyz="0.009320696924603175 7.83482142857143E-4 -0.026462549603174602"/>
+      </inertial>
+      <visual>
+        <geometry>
+          <mesh filename="package://${package_name}/meshes/kr10_r1100_2/visual/link_5.stl"/>
         </geometry>
         <origin rpy="-0.0 0.0 -0.0" xyz="0.0 0.0 0.0"/>
@@ -103,11 +129,16 @@
       <collision>
         <geometry>
-          <mesh filename="package://kuka_agilus_support/meshes/kr10_r1100_2/collision/link_6.stl"/>
-        </geometry>
-        <origin rpy="-0.0 0.0 -0.0" xyz="0.0 0.0 0.0"/>
-      </collision>
-      <visual>
-        <geometry>
-          <mesh filename="package://kuka_agilus_support/meshes/kr10_r1100_2/visual/link_6.stl"/>
+          <mesh filename="package://${package_name}/meshes/kr10_r1100_2/collision/link_6.stl"/>
+        </geometry>
+        <origin rpy="-0.0 0.0 -0.0" xyz="0.0 0.0 0.0"/>
+      </collision>
+      <inertial>
+        <inertia ixx="1.83698267603013E-4" ixy="0.0" ixz="0.0" iyy="1.8213621766783165E-4" iyz="0.0" izz="2.9589000000000004E-4"/>
+        <mass value="7.34E-1"/>
+        <origin rpy="0.0 -0.0 1.223427188696551" xyz="0.0 0.0 -0.011764604904632152"/>
+      </inertial>
+      <visual>
+        <geometry>
+          <mesh filename="package://${package_name}/meshes/kr10_r1100_2/visual/link_6.stl"/>
         </geometry>
         <origin rpy="-0.0 0.0 -0.0" xyz="0.0 0.0 0.0"/>

File: kuka_agilus_support/urdf/kr6_r700_sixx.urdf.xacro (robot description, xacro)
@@ -1,11 +1,16 @@
 <?xml version="1.0"?>
 <robot xmlns:xacro="http://www.ros.org/wiki/xacro" name="kr6_r700_sixx">
-  <!-- Import urdf file  -->
+  <!-- Import macro files  -->
   <xacro:include filename="$(find kuka_agilus_support)/urdf/kr6_r700_sixx_macro.xacro"/>
+  <xacro:include filename="$(find kuka_agilus_support)/urdf/kr_agilus_ros2_control_macro.xacro"/>
   <!-- Read additional arguments  -->
-  <xacro:arg name="use_fake_hardware" default="false"/>
+  <xacro:arg name="driver_version" default="rsi_only"/>
+  <xacro:arg name="mode" default="hardware"/>
+  <xacro:arg name="use_gpio" default="false"/>
   <xacro:arg name="roundtrip_time" default="0"/>
   <xacro:arg name="client_ip" default="0.0.0.0"/>
   <xacro:arg name="client_port" default="59152"/>
+  <xacro:arg name="controller_ip" default="0.0.0.0"/>
+  <xacro:arg name="verify_robot_model" default="true"/>
   <xacro:arg name="prefix" default=""/>
   <xacro:arg name="x" default="0"/>
@@ -15,5 +20,6 @@
   <xacro:arg name="pitch" default="0"/>
   <xacro:arg name="yaw" default="0"/>
-  <xacro:kuka_kr6_r700_sixx_robot client_ip="$(arg client_ip)" client_port="$(arg client_port)" prefix="$(arg prefix)" use_fake_hardware="$(arg use_fake_hardware)" roundtrip_time="$(arg roundtrip_time)">
+  <xacro:kuka_agilus_ros2_control name="$(arg prefix)kr6_r700_sixx" driver_version="$(arg driver_version)" client_ip="$(arg client_ip)" client_port="$(arg client_port)" controller_ip="$(arg controller_ip)" prefix="$(arg prefix)" mode="$(arg mode)" use_gpio="$(arg use_gpio)" roundtrip_time="$(arg roundtrip_time)" verify_robot_model="$(arg verify_robot_model)"/>
+  <xacro:kuka_kr6_r700_sixx_robot prefix="$(arg prefix)" package_name="kuka_agilus_support">
     <origin xyz="$(arg x) $(arg y) $(arg z)" rpy="$(arg roll) $(arg pitch) $(arg yaw)"/>
   </xacro:kuka_kr6_r700_sixx_robot>

File: kuka_agilus_support/urdf/kr6_r700_sixx_macro.xacro (robot description, xacro)
@@ -1,11 +1,9 @@
 <?xml version="1.0"?>
 <robot xmlns:xacro="http://wiki.ros.org/xacro">
+  <!-- include helper xacros -->
   <xacro:include filename="$(find kuka_resources)/urdf/common_constants.xacro"/>
   <xacro:include filename="$(find kuka_resources)/urdf/common_materials.xacro"/>
-  <xacro:include filename="$(find kuka_agilus_support)/urdf/kr_agilus_ros2_control.xacro"/>
-  <xacro:include filename="$(find kuka_agilus_support)/urdf/kr_agilus_transmission.xacro"/>
-  <xacro:macro name="kuka_kr6_r700_sixx_robot" params="client_ip client_port prefix use_fake_hardware roundtrip_time *origin">
-    <!-- ros2 control instance -->
-    <xacro:kuka_agilus_ros2_control name="${prefix}kr6_r700_sixx" client_ip="${client_ip}" client_port="${client_port}" prefix="${prefix}" use_fake_hardware="${use_fake_hardware}" roundtrip_time="${roundtrip_time}"/>
+  <xacro:macro name="kuka_kr6_r700_sixx_robot" params="prefix package_name *origin">
+    <!-- links - main serial chain -->
     <link name="world"/>
     <link name="${prefix}base_link">
@@ -13,5 +11,5 @@
         <origin xyz="0 0 0" rpy="0 0 0"/>
         <geometry>
-          <mesh filename="package://kuka_agilus_support/meshes/kr6_r700_sixx/visual/base_link.dae"/>
+          <mesh filename="package://${package_name}/meshes/kr6_r700_sixx/visual/base_link.dae"/>
         </geometry>
         <xacro:material_kuka_pedestal/>
@@ -20,5 +18,5 @@
         <origin xyz="0 0 0" rpy="0 0 0"/>
         <geometry>
-          <mesh filename="package://kuka_agilus_support/meshes/kr6_r700_sixx/collision/base_link.stl"/>
+          <mesh filename="package://${package_name}/meshes/kr6_r700_sixx/collision/base_link.stl"/>
         </geometry>
       </collision>
@@ -28,5 +26,5 @@
         <origin xyz="0 0 0" rpy="0 0 0"/>
         <geometry>
-          <mesh filename="package://kuka_agilus_support/meshes/kr6_r700_sixx/visual/link_1.dae"/>
+          <mesh filename="package://${package_name}/meshes/kr6_r700_sixx/visual/link_1.dae"/>
         </geometry>
         <xacro:material_kuka_orange/>
@@ -35,5 +33,5 @@
         <origin xyz="0 0 0" rpy="0 0 0"/>
         <geometry>
-          <mesh filename="package://kuka_agilus_support/meshes/kr6_r700_sixx/collision/link_1.stl"/>
+          <mesh filename="package://${package_name}/meshes/kr6_r700_sixx/collision/link_1.stl"/>
         </geometry>
       </collision>
@@ -43,5 +41,5 @@
         <origin xyz="0 0 0" rpy="0 0 0"/>
         <geometry>
-          <mesh filename="package://kuka_agilus_support/meshes/kr6_r700_sixx/visual/link_2.dae"/>
+          <mesh filename="package://${package_name}/meshes/kr6_r700_sixx/visual/link_2.dae"/>
         </geometry>
         <xacro:material_kuka_orange/>
@@ -50,5 +48,5 @@
         <origin xyz="0 0 0" rpy="0 0 0"/>
         <geometry>
-          <mesh filename="package://kuka_agilus_support/meshes/kr6_r700_sixx/collision/link_2.stl"/>
+          <mesh filename="package://${package_name}/meshes/kr6_r700_sixx/collision/link_2.stl"/>
         </geometry>
       </collision>
@@ -58,5 +56,5 @@
         <origin xyz="0 0 0" rpy="0 0 0"/>
         <geometry>
-          <mesh filename="package://kuka_agilus_support/meshes/kr6_r700_sixx/visual/link_3.dae"/>
+          <mesh filename="package://${package_name}/meshes/kr6_r700_sixx/visual/link_3.dae"/>
         </geometry>
         <xacro:material_kuka_orange/>
@@ -65,5 +63,5 @@
         <origin xyz="0 0 0" rpy="0 0 0"/>
         <geometry>
-          <mesh filename="package://kuka_agilus_support/meshes/kr6_r700_sixx/collision/link_3.stl"/>
+          <mesh filename="package://${package_name}/meshes/kr6_r700_sixx/collision/link_3.stl"/>
         </geometry>
       </collision>
@@ -73,5 +71,5 @@
         <origin xyz="0 0 0" rpy="0 0 0"/>
         <geometry>
-          <mesh filename="package://kuka_agilus_support/meshes/kr6_r700_sixx/visual/link_4.dae"/>
+          <mesh filename="package://${package_name}/meshes/kr6_r700_sixx/visual/link_4.dae"/>
         </geometry>
         <xacro:material_kuka_orange/>
@@ -80,5 +78,5 @@
         <origin xyz="0 0 0" rpy="0 0 0"/>
         <geometry>
-          <mesh filename="package://kuka_agilus_support/meshes/kr6_r700_sixx/collision/link_4.stl"/>
+          <mesh filename="package://${package_name}/meshes/kr6_r700_sixx/collision/link_4.stl"/>
         </geometry>
       </collision>
@@ -88,5 +86,5 @@
         <origin xyz="0 0 0" rpy="0 0 0"/>
         <geometry>
-          <mesh filename="package://kuka_agilus_support/meshes/kr6_r700_sixx/visual/link_5.dae"/>
+          <mesh filename="package://${package_name}/meshes/kr6_r700_sixx/visual/link_5.dae"/>
         </geometry>
         <xacro:material_kuka_orange/>
@@ -95,5 +93,5 @@
         <origin xyz="0 0 0" rpy="0 0 0"/>
         <geometry>
-          <mesh filename="package://kuka_agilus_support/meshes/kr6_r700_sixx/collision/link_5.stl"/>
+          <mesh filename="package://${package_name}/meshes/kr6_r700_sixx/collision/link_5.stl"/>
         </geometry>
       </collision>
@@ -103,5 +101,5 @@
         <origin xyz="0 0 0" rpy="0 0 0"/>
         <geometry>
-          <mesh filename="package://kuka_agilus_support/meshes/kr6_r700_sixx/visual/link_6.dae"/>
+          <mesh filename="package://${package_name}/meshes/kr6_r700_sixx/visual/link_6.dae"/>
         </geometry>
         <xacro:material_kuka_pedestal/>
@@ -110,5 +108,5 @@
         <origin xyz="0 0 0" rpy="0 0 0"/>
         <geometry>
-          <mesh filename="package://kuka_agilus_support/meshes/kr6_r700_sixx/collision/link_6.stl"/>
+          <mesh filename="package://${package_name}/meshes/kr6_r700_sixx/collision/link_6.stl"/>
         </geometry>
       </collision>

File: kuka_agilus_support/urdf/kr6_r900_sixx.urdf.xacro (robot description, xacro)
@@ -1,11 +1,16 @@
 <?xml version="1.0"?>
 <robot xmlns:xacro="http://www.ros.org/wiki/xacro" name="kr6_r900_sixx">
-  <!-- Import urdf file  -->
+  <!-- Import macro files  -->
   <xacro:include filename="$(find kuka_agilus_support)/urdf/kr6_r900_sixx_macro.xacro"/>
+  <xacro:include filename="$(find kuka_agilus_support)/urdf/kr_agilus_ros2_control_macro.xacro"/>
   <!-- Read additional arguments  -->
-  <xacro:arg name="use_fake_hardware" default="false"/>
+  <xacro:arg name="driver_version" default="rsi_only"/>
+  <xacro:arg name="mode" default="hardware"/>
+  <xacro:arg name="use_gpio" default="false"/>
   <xacro:arg name="roundtrip_time" default="0"/>
   <xacro:arg name="client_ip" default="0.0.0.0"/>
   <xacro:arg name="client_port" default="59152"/>
+  <xacro:arg name="controller_ip" default="0.0.0.0"/>
+  <xacro:arg name="verify_robot_model" default="true"/>
   <xacro:arg name="prefix" default=""/>
   <xacro:arg name="x" default="0"/>
@@ -15,5 +20,6 @@
   <xacro:arg name="pitch" default="0"/>
   <xacro:arg name="yaw" default="0"/>
-  <xacro:kuka_kr6_r900_sixx_robot client_ip="$(arg client_ip)" client_port="$(arg client_port)" prefix="$(arg prefix)" use_fake_hardware="$(arg use_fake_hardware)" roundtrip_time="$(arg roundtrip_time)">
+  <xacro:kuka_agilus_ros2_control name="$(arg prefix)kr6_r900_sixx" driver_version="$(arg driver_version)" client_ip="$(arg client_ip)" client_port="$(arg client_port)" controller_ip="$(arg controller_ip)" prefix="$(arg prefix)" mode="$(arg mode)" use_gpio="$(arg use_gpio)" roundtrip_time="$(arg roundtrip_time)" verify_robot_model="$(arg verify_robot_model)"/>
+  <xacro:kuka_kr6_r900_sixx_robot prefix="$(arg prefix)" package_name="kuka_agilus_support">
     <origin xyz="$(arg x) $(arg y) $(arg z)" rpy="$(arg roll) $(arg pitch) $(arg yaw)"/>
   </xacro:kuka_kr6_r900_sixx_robot>
