Commit message: Rebase from 'upstream'

File: kuka_agilus_support/urdf/kr6_r900_sixx_macro.xacro (robot description, xacro)
@@ -1,11 +1,9 @@
 <?xml version="1.0"?>
 <robot xmlns:xacro="http://wiki.ros.org/xacro">
+  <!-- include helper xacros -->
   <xacro:include filename="$(find kuka_resources)/urdf/common_constants.xacro"/>
   <xacro:include filename="$(find kuka_resources)/urdf/common_materials.xacro"/>
-  <xacro:include filename="$(find kuka_agilus_support)/urdf/kr_agilus_ros2_control.xacro"/>
-  <xacro:include filename="$(find kuka_agilus_support)/urdf/kr_agilus_transmission.xacro"/>
-  <xacro:macro name="kuka_kr6_r900_sixx_robot" params="client_ip client_port prefix use_fake_hardware roundtrip_time *origin">
-    <!-- ros2 control instance -->
-    <xacro:kuka_agilus_ros2_control name="${prefix}kr6_r900_sixx" client_ip="${client_ip}" client_port="${client_port}" prefix="${prefix}" use_fake_hardware="${use_fake_hardware}" roundtrip_time="${roundtrip_time}"/>
+  <xacro:macro name="kuka_kr6_r900_sixx_robot" params="prefix package_name *origin">
+    <!-- links - main serial chain -->
     <link name="world"/>
     <link name="${prefix}base_link">
@@ -13,5 +11,5 @@
         <origin xyz="0 0 0" rpy="0 0 0"/>
         <geometry>
-          <mesh filename="package://kuka_agilus_support/meshes/kr6_r900_sixx/visual/base_link.dae"/>
+          <mesh filename="package://${package_name}/meshes/kr6_r900_sixx/visual/base_link.dae"/>
         </geometry>
         <xacro:material_kuka_pedestal/>
@@ -20,5 +18,5 @@
         <origin xyz="0 0 0" rpy="0 0 0"/>
         <geometry>
-          <mesh filename="package://kuka_agilus_support/meshes/kr6_r900_sixx/collision/base_link.stl"/>
+          <mesh filename="package://${package_name}/meshes/kr6_r900_sixx/collision/base_link.stl"/>
         </geometry>
       </collision>
@@ -28,5 +26,5 @@
         <origin xyz="0 0 0" rpy="0 0 0"/>
         <geometry>
-          <mesh filename="package://kuka_agilus_support/meshes/kr6_r900_sixx/visual/link_1.dae"/>
+          <mesh filename="package://${package_name}/meshes/kr6_r900_sixx/visual/link_1.dae"/>
         </geometry>
         <xacro:material_kuka_orange/>
@@ -35,5 +33,5 @@
         <origin xyz="0 0 0" rpy="0 0 0"/>
         <geometry>
-          <mesh filename="package://kuka_agilus_support/meshes/kr6_r900_sixx/collision/link_1.stl"/>
+          <mesh filename="package://${package_name}/meshes/kr6_r900_sixx/collision/link_1.stl"/>
         </geometry>
       </collision>
@@ -43,5 +41,5 @@
         <origin xyz="0 0 0" rpy="0 0 0"/>
         <geometry>
-          <mesh filename="package://kuka_agilus_support/meshes/kr6_r900_sixx/visual/link_2.dae"/>
+          <mesh filename="package://${package_name}/meshes/kr6_r900_sixx/visual/link_2.dae"/>
         </geometry>
         <xacro:material_kuka_orange/>
@@ -50,5 +48,5 @@
         <origin xyz="0 0 0" rpy="0 0 0"/>
         <geometry>
-          <mesh filename="package://kuka_agilus_support/meshes/kr6_r900_sixx/collision/link_2.stl"/>
+          <mesh filename="package://${package_name}/meshes/kr6_r900_sixx/collision/link_2.stl"/>
         </geometry>
       </collision>
@@ -58,5 +56,5 @@
         <origin xyz="0 0 0" rpy="0 0 0"/>
         <geometry>
-          <mesh filename="package://kuka_agilus_support/meshes/kr6_r900_sixx/visual/link_3.dae"/>
+          <mesh filename="package://${package_name}/meshes/kr6_r900_sixx/visual/link_3.dae"/>
         </geometry>
         <xacro:material_kuka_orange/>
@@ -65,5 +63,5 @@
         <origin xyz="0 0 0" rpy="0 0 0"/>
         <geometry>
-          <mesh filename="package://kuka_agilus_support/meshes/kr6_r900_sixx/collision/link_3.stl"/>
+          <mesh filename="package://${package_name}/meshes/kr6_r900_sixx/collision/link_3.stl"/>
         </geometry>
       </collision>
@@ -73,5 +71,5 @@
         <origin xyz="0 0 0" rpy="0 0 0"/>
         <geometry>
-          <mesh filename="package://kuka_agilus_support/meshes/kr6_r900_sixx/visual/link_4.dae"/>
+          <mesh filename="package://${package_name}/meshes/kr6_r900_sixx/visual/link_4.dae"/>
         </geometry>
         <xacro:material_kuka_orange/>
@@ -80,5 +78,5 @@
         <origin xyz="0 0 0" rpy="0 0 0"/>
         <geometry>
-          <mesh filename="package://kuka_agilus_support/meshes/kr6_r900_sixx/collision/link_4.stl"/>
+          <mesh filename="package://${package_name}/meshes/kr6_r900_sixx/collision/link_4.stl"/>
         </geometry>
       </collision>
@@ -88,5 +86,5 @@
         <origin xyz="0 0 0" rpy="0 0 0"/>
         <geometry>
-          <mesh filename="package://kuka_agilus_support/meshes/kr6_r900_sixx/visual/link_5.dae"/>
+          <mesh filename="package://${package_name}/meshes/kr6_r900_sixx/visual/link_5.dae"/>
         </geometry>
         <xacro:material_kuka_orange/>
@@ -95,5 +93,5 @@
         <origin xyz="0 0 0" rpy="0 0 0"/>
         <geometry>
-          <mesh filename="package://kuka_agilus_support/meshes/kr6_r900_sixx/collision/link_5.stl"/>
+          <mesh filename="package://${package_name}/meshes/kr6_r900_sixx/collision/link_5.stl"/>
         </geometry>
       </collision>
@@ -103,5 +101,5 @@
         <origin xyz="0 0 0" rpy="0 0 0"/>
         <geometry>
-          <mesh filename="package://kuka_agilus_support/meshes/kr6_r900_sixx/visual/link_6.dae"/>
+          <mesh filename="package://${package_name}/meshes/kr6_r900_sixx/visual/link_6.dae"/>
         </geometry>
         <xacro:material_kuka_pedestal/>
@@ -110,5 +108,5 @@
         <origin xyz="0 0 0" rpy="0 0 0"/>
         <geometry>
-          <mesh filename="package://kuka_agilus_support/meshes/kr6_r900_sixx/collision/link_6.stl"/>
+          <mesh filename="package://${package_name}/meshes/kr6_r900_sixx/collision/link_6.stl"/>
         </geometry>
       </collision>

File: kuka_cybertech_support/urdf/kr16_r2010_2.urdf.xacro (robot description, xacro)
@@ -1,11 +1,16 @@
 <?xml version="1.0"?>
 <robot xmlns:xacro="http://www.ros.org/wiki/xacro" name="kr16_r2010_2">
-  <!-- Import urdf file  -->
+  <!-- Import macro files  -->
   <xacro:include filename="$(find kuka_cybertech_support)/urdf/kr16_r2010_2_macro.xacro"/>
+  <xacro:include filename="$(find kuka_cybertech_support)/urdf/kr_cybertech_ros2_control_macro.xacro"/>
   <!-- Read additional arguments  -->
-  <xacro:arg name="use_fake_hardware" default="false"/>
+  <xacro:arg name="driver_version" default="eki_rsi"/>
+  <xacro:arg name="mode" default="hardware"/>
+  <xacro:arg name="use_gpio" default="false"/>
   <xacro:arg name="roundtrip_time" default="0"/>
   <xacro:arg name="client_ip" default="0.0.0.0"/>
   <xacro:arg name="client_port" default="59152"/>
+  <xacro:arg name="controller_ip" default="0.0.0.0"/>
+  <xacro:arg name="verify_robot_model" default="true"/>
   <xacro:arg name="prefix" default=""/>
   <xacro:arg name="x" default="0"/>
@@ -15,5 +20,6 @@
   <xacro:arg name="pitch" default="0"/>
   <xacro:arg name="yaw" default="0"/>
-  <xacro:kuka_kr16_r2010_2_robot client_ip="$(arg client_ip)" client_port="$(arg client_port)" prefix="$(arg prefix)" use_fake_hardware="$(arg use_fake_hardware)" roundtrip_time="$(arg roundtrip_time)">
+  <xacro:kuka_cybertech_ros2_control name="$(arg prefix)kr16_r2010_2" driver_version="$(arg driver_version)" client_ip="$(arg client_ip)" client_port="$(arg client_port)" controller_ip="$(arg controller_ip)" prefix="$(arg prefix)" mode="$(arg mode)" use_gpio="$(arg use_gpio)" roundtrip_time="$(arg roundtrip_time)" verify_robot_model="$(arg verify_robot_model)"/>
+  <xacro:kuka_kr16_r2010_2_robot prefix="$(arg prefix)" package_name="kuka_cybertech_support">
     <origin xyz="$(arg x) $(arg y) $(arg z)" rpy="$(arg roll) $(arg pitch) $(arg yaw)"/>
   </xacro:kuka_kr16_r2010_2_robot>

File: kuka_cybertech_support/urdf/kr16_r2010_2_macro.xacro (robot description, xacro)
@@ -1,14 +1,11 @@
 <?xml version="1.0"?>
 <robot xmlns:xacro="http://wiki.ros.org/xacro">
-  <xacro:include filename="$(find kuka_cybertech_support)/urdf/kr_cybertech_ros2_control.xacro"/>
-  <xacro:include filename="$(find kuka_cybertech_support)/urdf/kr_cybertech_transmission.xacro"/>
-  <xacro:macro name="kuka_kr16_r2010_2_robot" params="client_ip client_port prefix use_fake_hardware roundtrip_time *origin">
-    <!-- ros2 control instance -->
-    <xacro:kuka_cybertech_ros2_control name="${prefix}kr16_r2010_2" client_ip="${client_ip}" client_port="${client_port}" prefix="${prefix}" use_fake_hardware="${use_fake_hardware}" roundtrip_time="${roundtrip_time}"/>
+  <xacro:macro name="kuka_kr16_r2010_2_robot" params="prefix package_name *origin">
+    <!-- links - main serial chain -->
     <link name="world"/>
     <link name="${prefix}base_link">
       <collision>
         <geometry>
-          <mesh filename="package://kuka_cybertech_support/meshes/kr16_r2010_2/collision/base_link.stl"/>
+          <mesh filename="package://${package_name}/meshes/kr16_r2010_2/collision/base_link.stl"/>
         </geometry>
         <origin rpy="-0.0 0.0 -0.0" xyz="0.0 0.0 0.0"/>
@@ -16,5 +13,5 @@
       <visual>
         <geometry>
-          <mesh filename="package://kuka_cybertech_support/meshes/kr16_r2010_2/visual/base_link.stl"/>
+          <mesh filename="package://${package_name}/meshes/kr16_r2010_2/visual/base_link.stl"/>
         </geometry>
         <origin rpy="-0.0 0.0 -0.0" xyz="0.0 0.0 0.0"/>
@@ -24,5 +21,5 @@
       <collision>
         <geometry>
-          <mesh filename="package://kuka_cybertech_support/meshes/kr16_r2010_2/collision/link_1.stl"/>
+          <mesh filename="package://${package_name}/meshes/kr16_r2010_2/collision/link_1.stl"/>
         </geometry>
         <origin rpy="-0.0 0.0 -0.0" xyz="0.0 0.0 0.0"/>
@@ -30,5 +27,5 @@
       <visual>
         <geometry>
-          <mesh filename="package://kuka_cybertech_support/meshes/kr16_r2010_2/visual/link_1.stl"/>
+          <mesh filename="package://${package_name}/meshes/kr16_r2010_2/visual/link_1.stl"/>
         </geometry>
         <origin rpy="-0.0 0.0 -0.0" xyz="0.0 0.0 0.0"/>
@@ -38,5 +35,5 @@
       <collision>
         <geometry>
-          <mesh filename="package://kuka_cybertech_support/meshes/kr16_r2010_2/collision/link_2.stl"/>
+          <mesh filename="package://${package_name}/meshes/kr16_r2010_2/collision/link_2.stl"/>
         </geometry>
         <origin rpy="-0.0 0.0 -0.0" xyz="0.0 0.0 0.0"/>
@@ -44,5 +41,5 @@
       <visual>
         <geometry>
-          <mesh filename="package://kuka_cybertech_support/meshes/kr16_r2010_2/visual/link_2.stl"/>
+          <mesh filename="package://${package_name}/meshes/kr16_r2010_2/visual/link_2.stl"/>
         </geometry>
         <origin rpy="-0.0 0.0 -0.0" xyz="0.0 0.0 0.0"/>
@@ -52,5 +49,5 @@
       <collision>
         <geometry>
-          <mesh filename="package://kuka_cybertech_support/meshes/kr16_r2010_2/collision/link_3.stl"/>
+          <mesh filename="package://${package_name}/meshes/kr16_r2010_2/collision/link_3.stl"/>
         </geometry>
         <origin rpy="-0.0 0.0 -0.0" xyz="0.0 0.0 0.0"/>
@@ -58,5 +55,5 @@
       <visual>
         <geometry>
-          <mesh filename="package://kuka_cybertech_support/meshes/kr16_r2010_2/visual/link_3.stl"/>
+          <mesh filename="package://${package_name}/meshes/kr16_r2010_2/visual/link_3.stl"/>
         </geometry>
         <origin rpy="-0.0 0.0 -0.0" xyz="0.0 0.0 0.0"/>
@@ -66,5 +63,5 @@
       <collision>
         <geometry>
-          <mesh filename="package://kuka_cybertech_support/meshes/kr16_r2010_2/collision/link_4.stl"/>
+          <mesh filename="package://${package_name}/meshes/kr16_r2010_2/collision/link_4.stl"/>
         </geometry>
         <origin rpy="-0.0 0.0 -0.0" xyz="0.0 0.0 0.0"/>
@@ -72,5 +69,5 @@
       <visual>
         <geometry>
-          <mesh filename="package://kuka_cybertech_support/meshes/kr16_r2010_2/visual/link_4.stl"/>
+          <mesh filename="package://${package_name}/meshes/kr16_r2010_2/visual/link_4.stl"/>
         </geometry>
         <origin rpy="-0.0 0.0 -0.0" xyz="0.0 0.0 0.0"/>
@@ -80,5 +77,5 @@
       <collision>
         <geometry>
-          <mesh filename="package://kuka_cybertech_support/meshes/kr16_r2010_2/collision/link_5.stl"/>
+          <mesh filename="package://${package_name}/meshes/kr16_r2010_2/collision/link_5.stl"/>
         </geometry>
         <origin rpy="-0.0 0.0 -0.0" xyz="0.0 0.0 0.0"/>
@@ -86,5 +83,5 @@
       <visual>
         <geometry>
-          <mesh filename="package://kuka_cybertech_support/meshes/kr16_r2010_2/visual/link_5.stl"/>
+          <mesh filename="package://${package_name}/meshes/kr16_r2010_2/visual/link_5.stl"/>
         </geometry>
         <origin rpy="-0.0 0.0 -0.0" xyz="0.0 0.0 0.0"/>
@@ -94,5 +91,5 @@
       <collision>
         <geometry>
-          <mesh filename="package://kuka_cybertech_support/meshes/kr16_r2010_2/collision/link_6.stl"/>
+          <mesh filename="package://${package_name}/meshes/kr16_r2010_2/collision/link_6.stl"/>
         </geometry>
         <origin rpy="-0.0 0.0 -0.0" xyz="0.0 0.0 0.0"/>
@@ -100,5 +97,5 @@
       <visual>
         <geometry>
-          <mesh filename="package://kuka_cybertech_support/meshes/kr16_r2010_2/visual/link_6.stl"/>
+          <mesh filename="package://${package_name}/meshes/kr16_r2010_2/visual/link_6.stl"/>
         </geometry>
         <origin rpy="-0.0 0.0 -0.0" xyz="0.0 0.0 0.0"/>
