Commit message: Rebase from 'release/humble/kuka_fortec_support'

File: urdf/kr240_r3330.urdf.xacro (robot description, xacro)
@@ -1,6 +1,6 @@
 <?xml version="1.0"?>
-<robot xmlns:xacro="http://www.ros.org/wiki/xacro" name="kr560_r3100_2">
+<robot xmlns:xacro="http://www.ros.org/wiki/xacro" name="kr240_r3330">
   <!-- Import macro files  -->
-  <xacro:include filename="$(find kuka_fortec_support)/urdf/kr560_r3100_2_macro.xacro"/>
+  <xacro:include filename="$(find kuka_fortec_support)/urdf/kr240_r3330_macro.xacro"/>
   <xacro:include filename="$(find kuka_fortec_support)/urdf/kr_fortec_ros2_control_macro.xacro"/>
   <!-- Read additional arguments  -->
@@ -20,7 +20,7 @@
   <xacro:arg name="pitch" default="0"/>
   <xacro:arg name="yaw" default="0"/>
-  <xacro:kuka_fortec_ros2_control name="$(arg prefix)kr560_r3100_2" driver_version="$(arg driver_version)" client_ip="$(arg client_ip)" client_port="$(arg client_port)" controller_ip="$(arg controller_ip)" prefix="$(arg prefix)" mode="$(arg mode)" use_gpio="$(arg use_gpio)" roundtrip_time="$(arg roundtrip_time)" verify_robot_model="$(arg verify_robot_model)"/>
-  <xacro:kuka_kr560_r3100_2_robot prefix="$(arg prefix)" package_name="kuka_fortec_support">
+  <xacro:kuka_fortec_ros2_control name="$(arg prefix)kr240_r3330" driver_version="$(arg driver_version)" client_ip="$(arg client_ip)" client_port="$(arg client_port)" controller_ip="$(arg controller_ip)" prefix="$(arg prefix)" mode="$(arg mode)" use_gpio="$(arg use_gpio)" roundtrip_time="$(arg roundtrip_time)" verify_robot_model="$(arg verify_robot_model)"/>
+  <xacro:kuka_kr240_r3330_robot prefix="$(arg prefix)" package_name="kuka_fortec_support">
     <origin xyz="$(arg x) $(arg y) $(arg z)" rpy="$(arg roll) $(arg pitch) $(arg yaw)"/>
-  </xacro:kuka_kr560_r3100_2_robot>
+  </xacro:kuka_kr240_r3330_robot>
 </robot>

File: urdf/kr_fortec_ros2_control_macro.xacro (robot description, xacro)
@@ -1,8 +1,14 @@
 <?xml version="1.0" encoding="UTF-8"?>
 <robot xmlns:xacro="http://www.ros.org/wiki/xacro">
-  <xacro:macro name="kuka_fortec_ros2_control" params="name client_ip client_port prefix use_fake_hardware roundtrip_time">
+  <xacro:macro name="kuka_fortec_ros2_control" params="name driver_version client_ip client_port controller_ip prefix mode use_gpio roundtrip_time verify_robot_model">
+    <!-- gazebo -->
+    <xacro:if value="${mode == 'gazebo'}">
+      <xacro:include filename="$(find kuka_gazebo)/gazebo/kuka_gazebo.xacro"/>
+      <xacro:kuka_gazebo controller_config_package="kuka_resources" controller_config_path="config/fake_hardware_config_6_axis.yaml"/>
+    </xacro:if>
+    <!-- ros2 control -->
     <ros2_control name="${name}" type="system">
       <hardware>
-        <xacro:if value="${use_fake_hardware}">
+        <xacro:if value="${mode == 'mock'}">
           <plugin>kuka_mock_hardware_interface::KukaMockHardwareInterface</plugin>
           <param name="cycle_time_ms">4</param>
@@ -11,9 +17,18 @@
           <param name="state_following_offset">0.0</param>
         </xacro:if>
-        <xacro:unless value="${use_fake_hardware}">
-          <plugin>kuka_kss_rsi_driver::KukaRSIHardwareInterface</plugin>
-          <param name="client_ip">${client_ip}</param>
-          <param name="client_port">${client_port}</param>
-        </xacro:unless>
+        <xacro:if value="${mode == 'hardware'}">
+          <xacro:if value="${driver_version == 'eki_rsi'}">
+            <plugin>kuka_rsi_driver::KukaEkiRsiHardwareInterface</plugin>
+            <param name="controller_ip">${controller_ip}</param>
+            <param name="name">${name}</param>
+            <param name="verify_robot_model">${verify_robot_model}</param>
+          </xacro:if>
+          <xacro:if value="${driver_version == 'rsi_only'}">
+            <plugin>kuka_rsi_driver::KukaRSIHardwareInterface</plugin>
+          </xacro:if>
+        </xacro:if>
+        <xacro:if value="${mode == 'gazebo'}">
+          <plugin>gz_ros2_control/GazeboSimSystem</plugin>
+        </xacro:if>
       </hardware>
       <joint name="${prefix}joint_1">
@@ -53,4 +68,11 @@
         </state_interface>
       </joint>
+      <xacro:if value="${use_gpio}">
+        <xacro:include filename="$(find kuka_rsi_driver)/config/gpio_config.xacro"/>
+        <xacro:gpio_config/>
+      </xacro:if>
+      <xacro:unless value="${use_gpio}">
+        <gpio name="gpio"/>
+      </xacro:unless>
     </ros2_control>
   </xacro:macro>
