Commit message: Rebase from 'release/humble/kuka_iontec_support'

File: urdf/kr_iontec_ros2_control_macro.xacro (robot description, xacro)
@@ -1,8 +1,14 @@
 <?xml version="1.0" encoding="UTF-8"?>
 <robot xmlns:xacro="http://www.ros.org/wiki/xacro">
-  <xacro:macro name="kuka_iontec_ros2_control" params="name client_ip client_port prefix use_fake_hardware roundtrip_time">
+  <xacro:macro name="kuka_iontec_ros2_control" params="name driver_version client_ip client_port controller_ip prefix mode use_gpio roundtrip_time verify_robot_model">
+    <!-- gazebo -->
+    <xacro:if value="${mode == 'gazebo'}">
+      <xacro:include filename="$(find kuka_gazebo)/gazebo/kuka_gazebo.xacro"/>
+      <xacro:kuka_gazebo controller_config_package="kuka_resources" controller_config_path="config/fake_hardware_config_6_axis.yaml"/>
+    </xacro:if>
+    <!-- ros2 control -->
     <ros2_control name="${name}" type="system">
       <hardware>
-        <xacro:if value="${use_fake_hardware}">
+        <xacro:if value="${mode == 'mock'}">
           <plugin>kuka_mock_hardware_interface::KukaMockHardwareInterface</plugin>
           <param name="cycle_time_ms">4</param>
@@ -11,9 +17,18 @@
           <param name="state_following_offset">0.0</param>
         </xacro:if>
-        <xacro:unless value="${use_fake_hardware}">
-          <plugin>kuka_kss_rsi_driver::KukaRSIHardwareInterface</plugin>
-          <param name="client_ip">${client_ip}</param>
-          <param name="client_port">${client_port}</param>
-        </xacro:unless>
+        <xacro:if value="${mode == 'hardware'}">
+          <xacro:if value="${driver_version == 'eki_rsi'}">
+            <plugin>kuka_rsi_driver::KukaEkiRsiHardwareInterface</plugin>
+            <param name="controller_ip">${controller_ip}</param>
+            <param name="name">${name}</param>
+            <param name="verify_robot_model">${verify_robot_model}</param>
+          </xacro:if>
+          <xacro:if value="${driver_version == 'rsi_only'}">
+            <plugin>kuka_rsi_driver::KukaRSIHardwareInterface</plugin>
+          </xacro:if>
+        </xacro:if>
+        <xacro:if value="${mode == 'gazebo'}">
+          <plugin>gz_ros2_control/GazeboSimSystem</plugin>
+        </xacro:if>
       </hardware>
       <joint name="${prefix}joint_1">
@@ -53,4 +68,11 @@
         </state_interface>
       </joint>
+      <xacro:if value="${use_gpio}">
+        <xacro:include filename="$(find kuka_rsi_driver)/config/gpio_config.xacro"/>
+        <xacro:gpio_config/>
+      </xacro:if>
+      <xacro:unless value="${use_gpio}">
+        <gpio name="gpio"/>
+      </xacro:unless>
     </ros2_control>
   </xacro:macro>
